File: schematic/lightcontroll/Power_management.sch (KiCad schematic (older format))
At the start: 26 parts, among them J14 ATX24connector, J15 PWR_JMP, J16 PWR_JMP, Q1 2N7000

Commit message: save Version 1.0
Parts:
- C10, C11, C14, C15, C18, C19, C22, C23: Mouser (none) -> https://www.mouser.de/ProductDetail/Wurth-Elektronik/885012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
- C12, C16, C20, C24: Mouser (none) -> https://www.mouser.de/ProductDetail/Murata-Electronics/GRM1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
- C13, C17, C21, C25, C26: Mouser (none) -> https://www.mouser.de/ProductDetail/Texas-Instruments/CD74H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
- D1: Mouser (none) -> https://www.mouser.de/ProductDetail/OSRAM-Opto-Semiconducto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
- J14: Mouser (none) -> https://www.mouser.de/ProductDetail/Molex/39-28-1243?qs=4XS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
- J17: renamed from J?; footprint (none) -> TerminalBlock_RND:TerminalBlock_RND_205-00295_1x10_P5.08mm_Horizontal; Mouser (none) -> https://www.reichelt.de/loetbare-schraubklemme-3-pol-rm-5-0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
- Q1: Mouser (none) -> https://www.mouser.de/ProductDetail/ON-Semiconductor/2N7000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
- R1: value 200 ohm -> 200
- R6: value 10k -> 10K
Connections:
- net GNDREF: now also J17.1 (Pin_1), J17.3 (Pin_3), J17.5 (Pin_5), J17.7 (Pin_7), J17.9 (Pin_9); no longer J17.10 (Pin_10), J17.2 (Pin_2), J17.4 (Pin_4), J17.6 (Pin_6), J17.8 (Pin_8)
- net 12V renamed +12V
- net +12V: now also J17.10 (Pin_10), J17.8 (Pin_8); no longer J17.1 (Pin_1), J17.3 (Pin_3)
- net 3V3 renamed +3V3
- net 5V renamed +5VD
- net +5VD: now also J17.2 (Pin_2), J17.4 (Pin_4), J17.6 (Pin_6); no longer J17.5 (Pin_5), J17.7 (Pin_7), J17.9 (Pin_9)
- net 5VSTANDBY renamed +5VL

Commit message: Updated PCB to Revision 2.0
- Added an 2.54mm pin header for second RS232 UART, which was already available in rev 1.0
- Changed all 2.00mm pin header to 2.54mm pin header. This fixes the mistake done in selecting the wrong footprint in rev 1.0
- Corrected schematic and layout of the spi to sk2812 circuits. During testing of previous rev some mistakes where found.
	* the second logical schemitac part of 74ls123 changes meaning of pin 6 and 7 compared to 15 and 14 of the first
	* The vibrator for the one signal needs to be also triggered with every rising edge, so use input A instead of binding it to gnd
	* Use the fourth nand to invert clock signal for a input of one vibrator
Parts:
- J15, J16: footprint Connector_PinHeader_2.00mm:PinHeader_1x02_P2.00mm_Vertical -> Connector_PinHeader_2.54mm:PinHeader_1x02_P2.54mm_Vertical
Changed lines of the file:
@@
 Title "ATX Power Supply connection"
 Date "2019-03-12"
-Rev "1.1"
+Rev "2.0"
 Comp "Tibersam Industries"
 Comment1 ""
@@
 F 0 "J15" H 2279 2792 50  0000 L CNN
 F 1 "PWR_JMP" H 2279 2701 50  0000 L CNN
-F 2 "Connector_PinHeader_2.00mm:PinHeader_1x02_P2.00mm_Vertical" H 2200 2800 50  0001 C CNN
+F 2 "Connector_PinHeader_2.54mm:PinHeader_1x02_P2.54mm_Vertical" H 2200 2800 50  0001 C CNN
 F 3 "~" H 2200 2800 50  0001 C CNN
 	1    2200 2800
@@
 F 0 "J16" H 2279 3792 50  0000 L CNN
 F 1 "PWR_JMP" H 2279 3701 50  0000 L CNN
-F 2 "Connector_PinHeader_2.00mm:PinHeader_1x02_P2.00mm_Vertical" H 2200 3800 50  0001 C CNN
+F 2 "Connector_PinHeader_2.54mm:PinHeader_1x02_P2.54mm_Vertical" H 2200 3800 50  0001 C CNN
 F 3 "~" H 2200 3800 50  0001 C CNN
 	1    2200 3800
