File: schematic/lightcontroll/lightcontroll.sch (KiCad schematic (older format))
At the start: 0 parts

Commit message: save before potential crash
Changed lines of the file:
@@
 $EndDescr
 $Sheet
-S 1600 1350 550  1300
+S 1600 1350 600  400
 U 5C818DF2
 F0 "stm32f407_blackboard" 50
 F1 "stm32f407blackboard.sch" 50
+F2 "5V" I L 1600 1450 50
+F3 "3.3V" I L 1600 1550 50
+F4 "5VSTANDBY" I L 1600 1650 50
+F5 "SPI" O R 2200 1450 50
+F6 "UART" O R 2200 1550 50
 $EndSheet
 $Sheet
@@
 $EndSheet
 $Sheet
-S 1900 3950 500  550
+S 1600 2100 500  550
 U 5C906D74
 F0 "UART Connections" 50
 F1 "uart_connections.sch" 50
+F2 "UART_IN" I L 1600 2150 50
 $EndSheet
+Text Label 2250 1550 0    50   ~ 0
+UART_5V
+Text Label 1250 2150 0    50   ~ 0
+UART_5V
+Wire Bus Line
+	2200 1550 2600 1550
+Wire Bus Line
+	1250 2150 1600 2150
 $EndSCHEMATC

Commit message: build backup
Changed lines of the file:
@@
 $EndDescr
 $Sheet
-S 1600 1350 600  400
+S 1600 1350 850  1150
 U 5C818DF2
 F0 "stm32f407_blackboard" 50
@@
 F3 "3.3V" I L 1600 1550 50
 F4 "5VSTANDBY" I L 1600 1650 50
-F5 "SPI" O R 2200 1450 50
-F6 "UART" O R 2200 1550 50
+F5 "SPI1" O R 2450 1450 50
+F6 "UART1" O R 2450 1550 50
+F7 "UART2" O R 2450 1650 50
+F8 "UART3" O R 2450 1750 50
+F9 "UART4" O R 2450 1850 50
+F10 "UART5" O R 2450 1950 50
+F11 "UART6" O R 2450 2050 50
+F12 "SPI2" O R 2450 2150 50
+F13 "SPI3" O R 2450 2250 50
 $EndSheet
 $Sheet
@@
 $EndSheet
 $Sheet
-S 1600 2100 500  550
+S 1600 2750 500  550
 U 5C906D74
 F0 "UART Connections" 50
 F1 "uart_connections.sch" 50
-F2 "UART_IN" I L 1600 2150 50
+F2 "UART_IN" I L 1600 2800 50
 $EndSheet
-Text Label 2250 1550 0    50   ~ 0
+Text Label 2500 1550 0    50   ~ 0
 UART_5V
-Text Label 1250 2150 0    50   ~ 0
+Text Label 1250 2800 0    50   ~ 0
 UART_5V
 Wire Bus Line
-	2200 1550 2600 1550
+	1250 2800 1600 2800
 Wire Bus Line
-	1250 2150 1600 2150
+	2450 1550 2850 1550
+Text Label 2500 1650 0    50   ~ 0
+UART2_5v
+Text Label 2500 1750 0    50   ~ 0
+UART3_5V
+Text Label 2500 1850 0    50   ~ 0
+UART4_5V
+Text Label 2500 1950 0    50   ~ 0
+UART5_5V
+Text Label 2500 2050 0    50   ~ 0
+UART6_5V
+Text Label 2500 2150 0    50   ~ 0
+SPI2
+Text Label 2500 2250 0    50   ~ 0
+SPI3
+Text Label 2500 1450 0    50   ~ 0
+SPI1
+Wire Bus Line
+	2450 1450 2850 1450
+Wire Bus Line
+	2450 1650 2850 1650
+Wire Bus Line
+	2450 1750 2850 1750
+Wire Bus Line
+	2450 1850 2850 1850
+Wire Bus Line
+	2450 1950 2850 1950
+Wire Bus Line
+	2450 2050 2850 2050
+Wire Bus Line
+	2450 2150 2850 2150
+Wire Bus Line
+	2450 2250 2850 2250
 $EndSCHEMATC

Commit message: save state
Changed lines of the file:
@@
 $Descr A4 11693 8268
 encoding utf-8
-Sheet 1 4
+Sheet 1 5
 Title ""
 Date ""
@@
 $EndSheet
 $Sheet
-S 4550 950  500  550
+S 4550 950  900  950
 U 5C8703FF
 F0 "ATX_Power" 50
 F1 "Power_management.sch" 50
-F2 "PS_ON" I L 4550 1050 50
-F3 "3.3V" O R 5050 1150 50
-F4 "5V" O R 5050 1250 50
-F5 "5VSTANDBY" O R 5050 1350 50
-F6 "PWR_OK" O R 5050 1450 50
+F2 "3.3V" O R 5450 1150 50
+F3 "5V" O R 5450 1250 50
+F4 "5VSTANDBY" O R 5450 1350 50
+F5 "PWR_OK" O R 5450 1450 50
+F6 "PS_ON_IN" I L 4550 1050 50
+F7 "12V" O R 5450 1050 50
 $EndSheet
 $Sheet
@@
 Wire Bus Line
 	2450 2250 2850 2250
+$Sheet
+S 1450 4000 550  650
+U 5C987024
+F0 "SPI_WS2812_DRIVERS" 50
+F1 "SPI_WS2812_DRIVERS.sch" 50
+$EndSheet
 $EndSCHEMATC
