File: schematic/lightcontroll/stm32f407blackboard.sch (KiCad schematic (older format))
At the start: 8 parts, among them J1 Header 16x2, J10 3.3V jumper, J2 Header 24x2, J3 Header 24X2

Commit message: save before potential crash
Parts:
- added J? (x2): UART/SPI JUMPER, symbol Connector_Generic:Conn_01x03
- added J?: UART3_JUMPER, symbol Connector_Generic:Conn_02x02_Counter_Clockwise
- added J?: UART/SPI JUMPER, symbol Connector_Generic:Conn_01x02
- added J?: UART5_JUMPER, symbol Connector_Generic:Conn_02x02_Counter_Clockwise
- added J?: UART1_JUMPER, symbol Connector_Generic:Conn_02x02_Counter_Clockwise
- added J?: Conn_02x02_Counter_Clockwise, symbol Connector_Generic:Conn_02x02_Counter_Clockwise
- added J?: UART2_JUMPER, symbol Connector_Generic:Conn_02x02_Counter_Clockwise
- added J? (x2): SPI_Jumper, symbol Connector_Generic_MountingPin:Conn_02x03_Odd_Even_MountingPin
Connections:
- net labels added: DATA0, DATA1, DATA2, DATAO, PA10, PA9, PC10_SPI, PC10_UART_TX, PC11_SPI, PC11_UART_RX, PC13_SPI, PCI10_SPI, SPI, SPI2, SPI3, UART, UART1, UART2, UART3, UART4, UART5, UART6
- net labels removed: MISO, MOSI, clk
- wire segments 322 -> 372
Other:
- note added: "CLK"
- note added: "RX"
- note added: "TX"
- note added: "UART4"
- note added: "clk"
- note removed: "SCK"

Commit message: build backup
Connections:
- net labels removed: SPI, UART
Changed lines of the file:
@@
 	1    0    0    -1
 $EndComp
-Entry Bus Bus
-	7400 1350 7500 1450
-Entry Bus Bus
-	7400 700  7500 800
-Entry Bus Bus
-	7400 1950 7500 2050
 Text Label 7200 700  0    50   ~ 0
 SPI1
@@
 Text Label 7200 1950 0    50   ~ 0
 SPI3
-Text HLabel 7600 800  2    50   Output ~ 0
-SPI
+Text HLabel 7400 700  2    50   Output ~ 0
+SPI1
 $Comp
 L Connector_Generic:Conn_01x03 J?
@@
 Text Label 9200 3400 0    50   ~ 0
 UART6
-Wire Bus Line
-	9400 2900 9150 2900
-Wire Bus Line
-	9400 3400 9150 3400
 Wire Wire Line
 	9050 2700 8750 2700
@@
 Wire Wire Line
 	6800 2600 6800 2650
-Wire Bus Line
-	7500 800  7600 800
 Wire Bus Line
 	7400 700  7150 700
@@
 Text Label 8850 3150 0    50   ~ 0
 DATA1
-Wire Bus Line
-	9150 2450 9400 2450
-Wire Bus Line
-	9150 2050 9400 2050
-Wire Bus Line
-	9150 1600 9400 1600
-Wire Bus Line
-	9150 1150 9400 1150
-Entry Bus Bus
-	9400 1150 9500 1250
-Entry Bus Bus
-	9400 1600 9500 1700
-Entry Bus Bus
-	9400 2050 9500 2150
-Entry Bus Bus
-	9400 2450 9500 2550
-Entry Bus Bus
-	9400 2900 9500 3000
-Entry Bus Bus
-	9400 3400 9500 3500
-Wire Bus Line
-	9500 900  9800 900
-Text HLabel 9800 900  2    50   Output ~ 0
-UART
+Text HLabel 9550 1150 2    50   Output ~ 0
+UART1
+Wire Bus Line
+	9150 1150 9550 1150
+Text HLabel 9550 1600 2    50   Output ~ 0
+UART2
+Wire Bus Line
+	9150 1600 9550 1600
+Text HLabel 9550 2050 2    50   Output ~ 0
+UART3
+Text HLabel 9550 2450 2    50   Output ~ 0
+UART4
+Text HLabel 9550 2900 2    50   Output ~ 0
+UART5
+Text HLabel 9550 3400 2    50   Output ~ 0
+UART6
+Wire Bus Line
+	9150 3400 9550 3400
+Wire Bus Line
+	9150 2900 9550 2900
+Wire Bus Line
+	9150 2450 9550 2450
+Wire Bus Line
+	9150 2050 9550 2050
+Text HLabel 7400 1350 2    50   Output ~ 0
+SPI2
+Text HLabel 7400 1950 2    50   Output ~ 0
+SPI3
 Wire Bus Line
 	9150 2700 9150 2900
@@
 	9150 1850 9150 2050
 Wire Bus Line
-	7500 800  7500 2050
-Wire Bus Line
 	7150 1950 7150 2150
 Wire Bus Line
@@
 Wire Bus Line
 	7150 700  7150 900
-Wire Bus Line
-	9500 900  9500 3500
 $EndSCHEMATC

Commit message: save state
Parts:
- removed J?: UART3_JUMPER, symbol Connector_Generic:Conn_02x02_Counter_Clockwise
- removed J?: UART5_JUMPER, symbol Connector_Generic:Conn_02x02_Counter_Clockwise
- removed J?: UART1_JUMPER, symbol Connector_Generic:Conn_02x02_Counter_Clockwise
- removed J?: Conn_02x02_Counter_Clockwise, symbol Connector_Generic:Conn_02x02_Counter_Clockwise
- removed J?: UART2_JUMPER, symbol Connector_Generic:Conn_02x02_Counter_Clockwise
- J1, J3: renamed from J?; footprint (none) -> Connector_PinHeader_2.54mm:PinHeader_2x03_P2.54mm_Vertical
- J10: renamed from J?; footprint (none) -> Connector_PinHeader_2.54mm:PinHeader_2x16_P2.54mm_Vertical
- J11: renamed from J10; footprint (none) -> Connector_PinHeader_2.54mm:PinHeader_1x02_P2.54mm_Vertical
- J12: renamed from J3; footprint (none) -> Connector_PinHeader_2.54mm:PinHeader_2x24_P2.54mm_Vertical
- J13: renamed from J?; footprint (none) -> Connector_PinHeader_2.54mm:PinHeader_2x24_P2.54mm_Vertical
- J2, J4, J5: renamed from J?; footprint (none) -> Connector_PinHeader_2.54mm:PinHeader_1x03_P2.54mm_Vertical
- J8: renamed from J?; footprint (none) -> Connector_PinHeader_2.54mm:PinHeader_1x02_P2.54mm_Vertical
- J9: renamed from J1; footprint (none) -> Connector_PinHeader_2.54mm:PinHeader_2x16_P2.54mm_Vertical
- gave numbers to parts that had none: 1
- renumbered J2 to J6
Connections:
- wire segments 372 -> 362
Other:
- note removed: "PA0/WK UP"
- note removed: "PA1"
- note removed: "PA10/RXD1"
- note removed: "PA11/USB_DM"
- note removed: "PA12/USB_DP"
- note removed: "PA15/TD1SWD"
- note removed: "PA2"
- note removed: "PA3"
- note removed: "PA4"
- note removed: "PA5"
- note removed: "PA6"
- note removed: "PA7"
- note removed: "PA8"
- note removed: "PA9/TXD1"
- note removed: "PB0"
- note removed: "PB1"
- note removed: "PB10"
- note removed: "PB11"
- note removed: "PB12"
- note removed: "PB13"
- note removed: "PB14"
- note removed: "PB3/TD0 SWD"
- note removed: "PB5"
- note removed: "PB6"
- note removed: "PB7"
- note removed: "PB8"
- note removed: "PB9"
- note removed: "PC0"
- note removed: "PC1"
- note removed: "PC10"
- note removed: "PC11"
- note removed: "PC12"
- note removed: "PC13"
- note removed: "PC2"
- note removed: "PC3"
- note removed: "PC4"
- note removed: "PC5"
- note removed: "PC6"
- note removed: "PC7"
- note removed: "PC8"
- note removed: "PC9"
- note removed: "PD0"
- note removed: "PD1"
- note removed: "PD10"
- note removed: "PD11"
- note removed: "PD12"
- note removed: "PD13"
- note removed: "PD14"
- note removed: "PD15"
- note removed: "PD2"
- note removed: "PD3"
- note removed: "PD4"
- note removed: "PD5"
- note removed: "PD6"
- note removed: "PD7"
- note removed: "PD8"
- note removed: "PD9"
- note removed: "PE0"
- note removed: "PE1"
- note removed: "PE10"
- note removed: "PE11"
- note removed: "PE12"
- note removed: "PE13"
- note removed: "PE14"
- note removed: "PE15"
- note removed: "PE2"
- note removed: "PE3"
- note removed: "PE4"
- note removed: "PE5"
- note removed: "PE6"
- note removed: "PE7"
- note removed: "PE8"
- note removed: "PE9"
- note removed: "VREF+"
- note removed: "VREF-"
