File: schematic/lightcontroll/stm32f407blackboard.sch (KiCad schematic (older format))
At the start: 18 parts, among them J1 SPI1_SS, J11 3.3V jumper, J12 Header 24X2, J13 Header 24X2, J2 5V Selector, J27 SPI1_MISO, J3 SPI1_CLK, J31 SPI1_MOSI, J33 SPI2_SS, J34 SPI2_CLK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

Commit message: save Version 1.0
Connections:
- no-connect marks 0 -> 2
Changed lines of the file:
@@
 Wire Wire Line
 	7200 3800 7700 3800
+Text HLabel 4300 2400 0    50   Input ~ 0
+PE2
+Text HLabel 4300 2500 0    50   Input ~ 0
+PE4
+Text HLabel 5400 2500 2    50   Output ~ 0
+PE5
+Text HLabel 4300 2600 0    50   Output ~ 0
+PE6
+NoConn ~ 8250 5000
+NoConn ~ 8200 4500
 $EndSCHEMATC
