File: schematic/lightcontroll/uart_connections.sch (KiCad schematic (older format))
At the start: 7 parts

Commit message: save before potential crash
Parts:
- added R?: R, symbol Device:R
- added U?: MAX13433EESD, Package_SO:SOIC-14_3.9x8.7mm_P1.27mm, symbol Interface_UART:MAX13433EESD
Connections:
- net labels added: RX1_IN, RX2_IN, TX1_OUT, TX2_OUT, UART1, UART2, UART_IN
- wire segments 17 -> 27
Changed lines of the file:
@@
 	4000 1750 3650 1750
 $Comp
-L power:+5V #PWR?
+L power:+5V #PWR0119
 U 1 1 5C907BCA
 P 3500 750
-F 0 "#PWR?" H 3500 600 50  0001 C CNN
+F 0 "#PWR0119" H 3500 600 50  0001 C CNN
 F 1 "+5V" H 3515 923 50  0000 C CNN
 F 2 "" H 3500 750 50  0001 C CNN
@@
 $EndComp
 $Comp
-L power:GNDREF #PWR?
+L power:GNDREF #PWR0120
 U 1 1 5C907C5E
 P 3750 1300
-F 0 "#PWR?" H 3750 1050 50  0001 C CNN
+F 0 "#PWR0120" H 3750 1050 50  0001 C CNN
 F 1 "GNDREF" V 3755 1172 50  0000 R CNN
 F 2 "" H 3750 1300 50  0001 C CNN
@@
 	3650 1950 3800 1950
 $Comp
-L power:GNDREF #PWR?
+L power:GNDREF #PWR0121
 U 1 1 5C90884B
 P 4250 1950
-F 0 "#PWR?" H 4250 1700 50  0001 C CNN
+F 0 "#PWR0121" H 4250 1700 50  0001 C CNN
 F 1 "GNDREF" V 4255 1822 50  0000 R CNN
 F 2 "" H 4250 1950 50  0001 C CNN
@@
 $EndComp
 $Comp
-L power:GNDREF #PWR?
+L power:GNDREF #PWR0122
 U 1 1 5C908864
 P 4250 2250
-F 0 "#PWR?" H 4250 2000 50  0001 C CNN
+F 0 "#PWR0122" H 4250 2000 50  0001 C CNN
 F 1 "GNDREF" V 4255 2122 50  0000 R CNN
 F 2 "" H 4250 2250 50  0001 C CNN
@@
 	4100 1950 4250 1950
 $Comp
-L power:GNDREF #PWR?
+L power:GNDREF #PWR0123
 U 1 1 5C9093B4
 P 2850 3550
-F 0 "#PWR?" H 2850 3300 50  0001 C CNN
+F 0 "#PWR0123" H 2850 3300 50  0001 C CNN
 F 1 "GNDREF" H 2855 3377 50  0000 C CNN
 F 2 "" H 2850 3550 50  0001 C CNN
@@
 	1    0    0    -1
 $EndComp
+Text GLabel 4200 2450 2    50   Output ~ 0
+TX1_OUT
+Wire Wire Line
+	4200 2450 3650 2450
+Text GLabel 4200 2650 2    50   Output ~ 0
+TX2_OUT
+Text GLabel 4200 2850 2    50   Input ~ 0
+RX1_IN
+Wire Wire Line
+	4200 2850 3650 2850
+Text GLabel 4200 3050 2    50   Input ~ 0
+RX2_IN
+Wire Wire Line
+	4200 3050 3650 3050
+Wire Wire Line
+	4200 2650 3650 2650
+Text HLabel 900  4150 0    50   Input ~ 0
+UART_IN
+Wire Bus Line
+	900  4150 1050 4150
+Wire Bus Line
+	1050 4150 1050 2750
+Wire Bus Line
+	1050 2750 1300 2750
+Entry Bus Bus
+	1300 2750 1400 2650
+Entry Bus Bus
+	1300 2750 1400 2850
+Wire Bus Line
+	1400 2650 1650 2650
+Wire Bus Line
+	1400 2850 1650 2850
+Text Label 1450 2650 0    50   ~ 0
+UART1
+Text Label 1450 2850 0    50   ~ 0
+UART2
+$Comp
+L Interface_UART:MAX13433EESD U?
+U 1 1 5C913A33
+P 2900 5550
+F 0 "U?" H 2900 6428 50  0000 C CNN
+F 1 "MAX13433EESD" H 2900 6337 50  0000 C CNN
+F 2 "Package_SO:SOIC-14_3.9x8.7mm_P1.27mm" H 2900 4550 50  0001 C CIN
+F 3 "https://datasheets.maximintegrated.com/en/ds/MAX13430E-MAX13433E.pdf" H 2900 6350 50  0001 C CNN
+	1    2900 5550
+	1    0    0    -1
+$EndComp
+$Comp
+L Device:R R?
+U 1 1 5C913BCB
+P 3700 5250
+F 0 "R?" H 3770 5296 50  0000 L CNN
+F 1 "R" H 3770 5205 50  0000 L CNN
+F 2 "" V 3630 5250 50  0001 C CNN
+F 3 "~" H 3700 5250 50  0001 C CNN
+	1    3700 5250
+	1    0    0    -1
+$EndComp
+Wire Wire Line
+	3400 5150 3550 5150
+Wire Wire Line
+	3550 5150 3550 5100
+Wire Wire Line
+	3550 5100 3700 5100
+Wire Wire Line
+	3700 5400 3550 5400
+Wire Wire Line
+	3550 5400 3550 5350
+Wire Wire Line
+	3550 5350 3400 5350
 $EndSCHEMATC

Commit message: build backup
Parts:
- added J?: RJ45_LED_Shielded, symbol Connector:RJ45_LED_Shielded
- added J?: DB9_Female_MountingHoles, symbol Connector:DB9_Female_MountingHoles
- added J?: UARTA, symbol Connector_Generic:Conn_02x03_Counter_Clockwise
- added J?: UARTB, symbol Connector_Generic:Conn_02x03_Counter_Clockwise
- added R?: R, symbol Device:R
- added U?: MAX13433EESD, Package_SO:SOIC-14_3.9x8.7mm_P1.27mm, symbol Interface_UART:MAX13433EESD
Connections:
- net labels added: DATA0, DATA1, UARTA_IN, UARTA_RS232_RX, UARTA_RS232_TX, UARTA_RS485_RX, UARTA_RS485_TX, UARTB_IN, UARTB_RS232_TX, UARTB_RS485_RX, UARTB_RX485_TX
- net labels removed: UART1, UART2, UART_IN
- wire segments 27 -> 86
Other:
- moved on the sheet: R?, U?

Commit message: save state
Parts:
- removed C? (x5): C, symbol Device:C
- added C2, C3: 1 uF, symbol Device:CP
- added C4, C5: 1 uF, symbol Device:CP_Small
- added C6: 1uF, symbol Device:C
- added C7: 100nF, symbol Device:C_Small
- added C8: 1uF, symbol Device:C_Small
- added C9: 100 nF, symbol Device:C_Small
- added J18: DB9_Female_MountingHoles, symbol Connector:DB9_Female_MountingHoles
- added J22: UARTB_TX_JMP, Connector_PinHeader_2.00mm:PinHeader_2x03_P2.00mm_Vertical, symbol Connector_Generic:Conn_02x03_Counter_Clockwise
- added J23: UARTB_RX_JMP, Connector_PinHeader_2.00mm:PinHeader_2x03_P2.00mm_Vertical, symbol Connector_Generic:Conn_02x03_Counter_Clockwise
- added J24: UART_RX_JMP, Connector_PinHeader_2.00mm:PinHeader_2x03_P2.00mm_Vertical, symbol Connector_Generic:Conn_02x03_Counter_Clockwise
- added J25: UARTA_TX_JMP, Connector_PinHeader_2.00mm:PinHeader_2x03_P2.00mm_Vertical, symbol Connector_Generic:Conn_02x03_Counter_Clockwise
- added R3, R4: R, symbol Device:R
- C1: renamed from C?; value CP -> 1 uF
- J19, J20: renamed from J?; footprint (none) -> Connector_PinHeader_2.00mm:PinHeader_2x03_P2.00mm_Vertical
- R2: renamed from R?; value R -> 120 Ohm
- gave numbers to parts that had none: 6
Connections:
- net labels added: UARTA_RX_EN, UARTA_RX_EN_JMP, UARTA_TX_EN, UARTA_TX_EN_JMP, UARTB_RS232_RX, UARTB_RX_EN, UARTB_RX_EN_JMP, UARTB_TX_EN, UARTB_TX_EN_JMP, UART_RX_EN_JMP, UART_TX_EN_JMP, VCC, uartb_rx-, uartb_tx+, uartb_tx-, vcc
- net labels removed: +5V, RX1_IN, RX2_IN, TX1_OUT, TX2_OUT
- wire segments 86 -> 147
- no-connect marks 0 -> 9
Other:
- moved on the sheet: J17
