File: schematic/lightcontroll/uart_connections.sch (KiCad schematic (older format))
At the start: 19 parts, among them J21 RJ45_LED_Shielded, J22 Conn_01x03, J23 Conn_01x03, J24 Conn_01x03, J25 Conn_01x03, J37 Conn_01x03, J38 Conn_01x03, J39 Conn_01x03, J40 Conn_01x03, U2 MAX13433EESD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

Commit message: save Version 1.0
Parts:
- C6, C7, C8: Mouser (none) -> https://www.mouser.de/ProductDetail/Wurth-Elektronik/885012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
- C9: value 100 nF -> 100nF; Mouser (none) -> https://www.mouser.de/ProductDetail/Wurth-Elektronik/885012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
- J21: Mouser (none) -> https://www.mouser.de/ProductDetail/Stewart-Connector-Bel/S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
- R2: value 120 Ohm -> 120
- R3, R4: value R -> 200
- R5: value R -> 120
- U2, U3: Mouser (none) -> https://www.mouser.de/ProductDetail/Maxim-Integrated/MAX134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
Changed lines of the file:
@@
 F 2 "Package_SO:SOIC-14_3.9x8.7mm_P1.27mm" H 2500 5900 50  0001 C CIN
 F 3 "https://datasheets.maximintegrated.com/en/ds/MAX13430E-MAX13433E.pdf" H 2500 7700 50  0001 C CNN
+F 4 "https://www.mouser.de/ProductDetail/Maxim-Integrated/MAX13433EESD%2b?qs=CDqwynd4ZNpm7OXRo1qQYw%3D%3D" H 2500 6900 50  0001 C CNN "Mouser"
 	1    2500 6900
 	1    0    0    -1
@@
 P 3300 6600
 F 0 "R5" H 3370 6646 50  0000 L CNN
-F 1 "R" H 3370 6555 50  0000 L CNN
+F 1 "120" H 3370 6555 50  0000 L CNN
 F 2 "Resistor_SMD:R_0603_1608Metric_Pad1.05x0.95mm_HandSolder" V 3230 6600 50  0001 C CNN
 F 3 "~" H 3300 6600 50  0001 C CNN
@@
 F 2 "Connector_RJ:RJ45_BEL_SS74301-00x_Vertical" V 6050 6175 50  0001 C CNN
 F 3 "~" V 6050 6175 50  0001 C CNN
+F 4 "https://www.mouser.de/ProductDetail/Stewart-Connector-Bel/SS-74301-001?qs=%2Fha2pyFadugHtoWXbf7rjzodwtXlWR8vdipjKL0ybnsmrvyKMPQLNw%3D%3D" H 6050 6150 50  0001 C CNN "Mouser"
 	1    6050 6150
 	-1   0    0    1
@@
 F 2 "Package_SO:SOIC-14_3.9x8.7mm_P1.27mm" H 3000 4100 50  0001 C CIN
 F 3 "https://datasheets.maximintegrated.com/en/ds/MAX13430E-MAX13433E.pdf" H 3000 5900 50  0001 C CNN
+F 4 "https://www.mouser.de/ProductDetail/Maxim-Integrated/MAX13433EESD%2b?qs=CDqwynd4ZNpm7OXRo1qQYw%3D%3D" H 3000 5100 50  0001 C CNN "Mouser"
 	1    3000 5100
 	1    0    0    -1
@@
 P 3700 4750
 F 0 "R2" H 3770 4796 50  0000 L CNN
-F 1 "120 Ohm" H 3770 4705 50  0000 L CNN
+F 1 "120" H 3770 4705 50  0000 L CNN
 F 2 "Resistor_SMD:R_0603_1608Metric_Pad1.05x0.95mm_HandSolder" V 3630 4750 50  0001 C CNN
 F 3 "~" H 3700 4750 50  0001 C CNN
@@
 F 2 "Capacitor_SMD:C_0603_1608Metric_Pad1.05x0.95mm_HandSolder" H 3788 4250 50  0001 C CNN
 F 3 "~" H 3750 4400 50  0001 C CNN
+F 4 "https://www.mouser.de/ProductDetail/Wurth-Elektronik/885012206052?qs=0KOYDY2FL2%2F2JKabApojcQ%3D%3D" H 3750 4400 50  0001 C CNN "Mouser"
 	1    3750 4400
 	1    0    0    -1
@@
 F 2 "Capacitor_SMD:C_0603_1608Metric_Pad1.05x0.95mm_HandSolder" H 2200 4600 50  0001 C CNN
 F 3 "~" H 2200 4600 50  0001 C CNN
+F 4 "https://www.mouser.de/ProductDetail/Wurth-Elektronik/885012206071?qs=0KOYDY2FL2%2FEBQkuHgvarg%3D%3D" H 2200 4600 50  0001 C CNN "Mouser"
 	1    2200 4600
 	0    1    1    0
@@
 F 2 "Capacitor_SMD:C_0603_1608Metric_Pad1.05x0.95mm_HandSolder" H 3050 6200 50  0001 C CNN
 F 3 "~" H 3050 6200 50  0001 C CNN
+F 4 "https://www.mouser.de/ProductDetail/Wurth-Elektronik/885012206052?qs=0KOYDY2FL2%2F2JKabApojcQ%3D%3D" H 3050 6200 50  0001 C CNN "Mouser"
 	1    3050 6200
 	1    0    0    -1
@@
 P 1750 6400
 F 0 "C9" V 1521 6400 50  0000 C CNN
-F 1 "100 nF" V 1612 6400 50  0000 C CNN
+F 1 "100nF" V 1612 6400 50  0000 C CNN
 F 2 "Capacitor_SMD:C_0603_1608Metric_Pad1.05x0.95mm_HandSolder" H 1750 6400 50  0001 C CNN
 F 3 "~" H 1750 6400 50  0001 C CNN
+F 4 "https://www.mouser.de/ProductDetail/Wurth-Elektronik/885012206071?qs=0KOYDY2FL2%2FEBQkuHgvarg%3D%3D" H 1750 6400 50  0001 C CNN "Mouser"
 	1    1750 6400
 	0    1    1    0
@@
 P 6550 5700
 F 0 "R3" H 6620 5746 50  0000 L CNN
-F 1 "R" H 6620 5655 50  0000 L CNN
+F 1 "200" H 6620 5655 50  0000 L CNN
 F 2 "Resistor_SMD:R_0603_1608Metric_Pad1.05x0.95mm_HandSolder" V 6480 5700 50  0001 C CNN
 F 3 "~" H 6550 5700 50  0001 C CNN
@@
 P 6650 6450
 F 0 "R4" V 6443 6450 50  0000 C CNN
-F 1 "R" V 6534 6450 50  0000 C CNN
+F 1 "200" V 6534 6450 50  0000 C CNN
 F 2 "Resistor_SMD:R_0603_1608Metric_Pad1.05x0.95mm_HandSolder" V 6580 6450 50  0001 C CNN
 F 3 "~" H 6650 6450 50  0001 C CNN
@@
 UARTA_TX_N
 $Comp
-L power:GNDREF #PWR?
+L power:GNDREF #PWR0108
 U 1 1 5ED7AAC4
 P 6050 5650
-F 0 "#PWR?" H 6050 5400 50  0001 C CNN
+F 0 "#PWR0108" H 6050 5400 50  0001 C CNN
 F 1 "GNDREF" H 6055 5477 50  0000 C CNN
 F 2 "" H 6050 5650 50  0001 C CNN
